File: plant-watering/Relais.sch (KiCad schematic (older format))
At the start: 6 parts, among them K1 HJR-4102-L-05V, K2 HJR-4102-L-05V, K3 HJR-4102-L-05V

Commit message: changed transistor and relay circuit
Parts:
- K1, K2, K3: symbol HJR-4102-L-05V:HJR-4102-L-05V -> plant-watering-rescue:HJR-4102-L-05V-HJR-4102-L-05V
Connections:
- net labels removed: GND
- wire segments 31 -> 27
Changed lines of the file:
@@
 $EndDescr
 $Comp
-L HJR-4102-L-05V:HJR-4102-L-05V K2
+L plant-watering-rescue:HJR-4102-L-05V-HJR-4102-L-05V K2
 U 1 1 600A0827
 P 6000 3450
+AR Path="/600A0827" Ref="K2"  Part="1"
+AR Path="/600A014F/600A0827" Ref="K2"  Part="1"
 F 0 "K2" H 6000 3917 50  0000 C CNN
 F 1 "HJR-4102-L-05V" H 6000 3826 50  0000 C CNN
@@
 $EndComp
 $Comp
-L HJR-4102-L-05V:HJR-4102-L-05V K1
+L plant-watering-rescue:HJR-4102-L-05V-HJR-4102-L-05V K1
 U 1 1 600A2E74
 P 4250 3450
+AR Path="/600A2E74" Ref="K1"  Part="1"
+AR Path="/600A014F/600A2E74" Ref="K1"  Part="1"
 F 0 "K1" H 4250 3917 50  0000 C CNN
 F 1 "HJR-4102-L-05V" H 4250 3826 50  0000 C CNN
@@
 $EndComp
 $Comp
-L HJR-4102-L-05V:HJR-4102-L-05V K3
+L plant-watering-rescue:HJR-4102-L-05V-HJR-4102-L-05V K3
 U 1 1 600A5240
 P 7800 3450
+AR Path="/600A5240" Ref="K3"  Part="1"
+AR Path="/600A014F/600A5240" Ref="K3"  Part="1"
 F 0 "K3" H 7800 3917 50  0000 C CNN
 F 1 "HJR-4102-L-05V" H 7800 3826 50  0000 C CNN
@@
 F 7 "Manufacturer Recommendations" H 7800 3450 50  0001 L BNN "STANDARD"
 	1    7800 3450
-	1    0    0    -1
-$EndComp
-Wire Wire Line
-	3850 3650 3850 4050
-Wire Wire Line
-	5600 3650 5600 4050
-Wire Wire Line
-	5600 4050 3850 4050
-Wire Wire Line
-	7400 3650 7400 4050
-Wire Wire Line
-	7400 4050 5600 4050
-Connection ~ 5600 4050
-Wire Wire Line
-	3850 4050 3600 4050
-Wire Wire Line
-	3600 4050 3600 4100
-Connection ~ 3850 4050
-$Comp
-L power:GND #PWR0105
-U 1 1 600A6335
-P 3600 4100
-F 0 "#PWR0105" H 3600 3850 50  0001 C CNN
-F 1 "GND" H 3605 3927 50  0000 C CNN
-F 2 "" H 3600 4100 50  0001 C CNN
-F 3 "" H 3600 4100 50  0001 C CNN
-	1    3600 4100
 	1    0    0    -1
 $EndComp
@@
 	8300 3450 8300 2750
 Wire Wire Line
-	8300 2750 6500 2750
+	8300 2750 7250 2750
 Wire Wire Line
 	6400 3450 6500 3450
@@
 Connection ~ 6500 2750
 Wire Wire Line
-	6500 2750 4750 2750
+	6500 2750 5500 2750
 Wire Wire Line
 	4650 3450 4750 3450
@@
 Connection ~ 4750 2750
 Wire Wire Line
-	4750 2750 3600 2750
+	4750 2750 3750 2750
 Text GLabel 4650 3650 2    50   Input ~ 0
 M1
@@
 Text GLabel 8200 3650 2    50   Input ~ 0
 M3
-Text GLabel 3650 3250 0    50   Input ~ 0
+Text GLabel 3750 3650 0    50   Input ~ 0
 RelayS1
-Text GLabel 5400 3250 0    50   Input ~ 0
+Text GLabel 5500 3650 0    50   Input ~ 0
 RelayS2
-Text GLabel 7200 3250 0    50   Input ~ 0
+Text GLabel 7250 3650 0    50   Input ~ 0
 RelayS3
 $Comp
@@
 $EndComp
 Wire Wire Line
-	3650 3250 3750 3250
-Wire Wire Line
 	3750 3300 3750 3250
-Connection ~ 3750 3250
 Wire Wire Line
 	3750 3250 3850 3250
@@
 Wire Wire Line
 	3750 3650 3850 3650
-Connection ~ 3850 3650
 Wire Wire Line
 	5500 3600 5500 3650
 Wire Wire Line
 	5500 3650 5600 3650
-Connection ~ 5600 3650
 Wire Wire Line
 	5600 3250 5500 3250
 Wire Wire Line
 	5500 3300 5500 3250
-Connection ~ 5500 3250
-Wire Wire Line
-	5500 3250 5400 3250
-Wire Wire Line
-	7200 3250 7250 3250
 Wire Wire Line
 	7250 3250 7250 3300
-Connection ~ 7250 3250
 Wire Wire Line
 	7250 3250 7400 3250
@@
 Wire Wire Line
 	7250 3650 7400 3650
-Connection ~ 7400 3650
+Wire Wire Line
+	3750 3250 3750 2750
+Connection ~ 3750 3250
+Connection ~ 3750 2750
+Wire Wire Line
+	3750 2750 3600 2750
+Wire Wire Line
+	5500 3250 5500 2750
+Connection ~ 5500 3250
+Connection ~ 5500 2750
+Wire Wire Line
+	5500 2750 4750 2750
+Wire Wire Line
+	7250 3250 7250 2750
+Connection ~ 7250 3250
+Connection ~ 7250 2750
+Wire Wire Line
+	7250 2750 6500 2750
 $EndSCHEMATC

Commit message: edited schematic & started pcb design
Parts:
- removed K1, K2, K3: HJR-4102-L-05V, HJR-4102-L-05V:RELAY_HJR-4102-L-05V, symbol plant-watering-rescue:HJR-4102-L-05V-HJR-4102-L-05V
- added K1, K2, K3: SRD-05VDC-SL-C, SRD-05VDC-SL-C:RELAY_SRD-05VDC-SL-C, symbol SRD-05VDC-SL-C:SRD-05VDC-SL-C
- D1, D2, D3: footprint (none) -> Diodes_ThroughHole:D_DO-41_SOD81_P7.62mm_Horizontal
Connections:
- wire segments 27 -> 24
Changed lines of the file:
@@
 $EndDescr
-$Comp
-L plant-watering-rescue:HJR-4102-L-05V-HJR-4102-L-05V K2
-U 1 1 600A0827
-P 6000 3450
-AR Path="/600A0827" Ref="K2"  Part="1"
-AR Path="/600A014F/600A0827" Ref="K2"  Part="1"
-F 0 "K2" H 6000 3917 50  0000 C CNN
-F 1 "HJR-4102-L-05V" H 6000 3826 50  0000 C CNN
-F 2 "HJR-4102-L-05V:RELAY_HJR-4102-L-05V" H 6000 3450 50  0001 L BNN
-F 3 "" H 6000 3450 50  0001 L BNN
-F 4 "Tianbo Electronics" H 6000 3450 50  0001 L BNN "MANUFACTURER"
-F 5 "11.70 mm" H 6000 3450 50  0001 L BNN "MAXIMUM_PACKAGE_HEIGHT"
-F 6 "N/A" H 6000 3450 50  0001 L BNN "PARTREV"
-F 7 "Manufacturer Recommendations" H 6000 3450 50  0001 L BNN "STANDARD"
-	1    6000 3450
-	1    0    0    -1
-$EndComp
-$Comp
-L plant-watering-rescue:HJR-4102-L-05V-HJR-4102-L-05V K1
-U 1 1 600A2E74
-P 4250 3450
-AR Path="/600A2E74" Ref="K1"  Part="1"
-AR Path="/600A014F/600A2E74" Ref="K1"  Part="1"
-F 0 "K1" H 4250 3917 50  0000 C CNN
-F 1 "HJR-4102-L-05V" H 4250 3826 50  0000 C CNN
-F 2 "HJR-4102-L-05V:RELAY_HJR-4102-L-05V" H 4250 3450 50  0001 L BNN
-F 3 "" H 4250 3450 50  0001 L BNN
-F 4 "Tianbo Electronics" H 4250 3450 50  0001 L BNN "MANUFACTURER"
-F 5 "11.70 mm" H 4250 3450 50  0001 L BNN "MAXIMUM_PACKAGE_HEIGHT"
-F 6 "N/A" H 4250 3450 50  0001 L BNN "PARTREV"
-F 7 "Manufacturer Recommendations" H 4250 3450 50  0001 L BNN "STANDARD"
-	1    4250 3450
-	1    0    0    -1
-$EndComp
-$Comp
-L plant-watering-rescue:HJR-4102-L-05V-HJR-4102-L-05V K3
-U 1 1 600A5240
-P 7800 3450
-AR Path="/600A5240" Ref="K3"  Part="1"
-AR Path="/600A014F/600A5240" Ref="K3"  Part="1"
-F 0 "K3" H 7800 3917 50  0000 C CNN
-F 1 "HJR-4102-L-05V" H 7800 3826 50  0000 C CNN
-F 2 "HJR-4102-L-05V:RELAY_HJR-4102-L-05V" H 7800 3450 50  0001 L BNN
-F 3 "" H 7800 3450 50  0001 L BNN
-F 4 "Tianbo Electronics" H 7800 3450 50  0001 L BNN "MANUFACTURER"
-F 5 "11.70 mm" H 7800 3450 50  0001 L BNN "MAXIMUM_PACKAGE_HEIGHT"
-F 6 "N/A" H 7800 3450 50  0001 L BNN "PARTREV"
-F 7 "Manufacturer Recommendations" H 7800 3450 50  0001 L BNN "STANDARD"
-	1    7800 3450
-	1    0    0    -1
-$EndComp
 $Comp
 L power:+5V #PWR0106
@@
 	1    0    0    -1
 $EndComp
-Wire Wire Line
-	8200 3450 8300 3450
-Wire Wire Line
-	8300 3450 8300 2750
-Wire Wire Line
-	8300 2750 7250 2750
-Wire Wire Line
-	6400 3450 6500 3450
-Wire Wire Line
-	6500 3450 6500 2750
-Connection ~ 6500 2750
-Wire Wire Line
-	6500 2750 5500 2750
-Wire Wire Line
-	4650 3450 4750 3450
-Wire Wire Line
-	4750 3450 4750 2750
-Connection ~ 4750 2750
-Wire Wire Line
-	4750 2750 3750 2750
-Text GLabel 4650 3650 2    50   Input ~ 0
+Text GLabel 4550 3400 2    50   Input ~ 0
 M1
-Text GLabel 6400 3650 2    50   Input ~ 0
+Text GLabel 6300 3400 2    50   Input ~ 0
 M2
-Text GLabel 8200 3650 2    50   Input ~ 0
+Text GLabel 8100 3400 2    50   Input ~ 0
 M3
 Text GLabel 3750 3650 0    50   Input ~ 0
@@
 F 0 "D1" V 3704 3530 50  0000 L CNN
 F 1 "D" V 3795 3530 50  0000 L CNN
-F 2 "" H 3750 3450 50  0001 C CNN
+F 2 "Diodes_ThroughHole:D_DO-41_SOD81_P7.62mm_Horizontal" H 3750 3450 50  0001 C CNN
 F 3 "~" H 3750 3450 50  0001 C CNN
 	1    3750 3450
@@
 F 0 "D2" V 5454 3530 50  0000 L CNN
 F 1 "D" V 5545 3530 50  0000 L CNN
-F 2 "" H 5500 3450 50  0001 C CNN
+F 2 "Diodes_ThroughHole:D_DO-41_SOD81_P7.62mm_Horizontal" H 5500 3450 50  0001 C CNN
 F 3 "~" H 5500 3450 50  0001 C CNN
 	1    5500 3450
@@
 F 0 "D3" V 7204 3530 50  0000 L CNN
 F 1 "D" V 7295 3530 50  0000 L CNN
-F 2 "" H 7250 3450 50  0001 C CNN
+F 2 "Diodes_ThroughHole:D_DO-41_SOD81_P7.62mm_Horizontal" H 7250 3450 50  0001 C CNN
 F 3 "~" H 7250 3450 50  0001 C CNN
 	1    7250 3450
@@
 $EndComp
 Wire Wire Line
-	3750 3300 3750 3250
-Wire Wire Line
-	3750 3250 3850 3250
-Wire Wire Line
 	3750 3600 3750 3650
-Wire Wire Line
-	3750 3650 3850 3650
 Wire Wire Line
 	5500 3600 5500 3650
 Wire Wire Line
-	5500 3650 5600 3650
-Wire Wire Line
-	5600 3250 5500 3250
-Wire Wire Line
-	5500 3300 5500 3250
-Wire Wire Line
-	7250 3250 7250 3300
-Wire Wire Line
-	7250 3250 7400 3250
-Wire Wire Line
 	7250 3600 7250 3650
-Wire Wire Line
-	7250 3650 7400 3650
-Wire Wire Line
-	3750 3250 3750 2750
-Connection ~ 3750 3250
 Connection ~ 3750 2750
 Wire Wire Line
 	3750 2750 3600 2750
+Connection ~ 5500 2750
+Connection ~ 7250 2750
+$Comp
+L SRD-05VDC-SL-C:SRD-05VDC-SL-C K1
+U 1 1 600B0E95
+P 4250 3400
+F 0 "K1" H 4250 3767 50  0000 C CNN
+F 1 "SRD-05VDC-SL-C" H 4250 3676 50  0000 C CNN
+F 2 "SRD-05VDC-SL-C:RELAY_SRD-05VDC-SL-C" H 4250 3400 50  0001 L BNN
+F 3 "" H 4250 3400 50  0001 L BNN
+F 4 "IPC-7251" H 4250 3400 50  0001 L BNN "STANDARD"
+F 5 "SONGLE RELAY" H 4250 3400 50  0001 L BNN "MANUFACTURER"
+	1    4250 3400
+	1    0    0    -1
+$EndComp
 Wire Wire Line
-	5500 3250 5500 2750
-Connection ~ 5500 3250
-Connection ~ 5500 2750
+	3750 2750 3750 3300
 Wire Wire Line
-	5500 2750 4750 2750
+	3750 2750 4650 2750
+$Comp
+L SRD-05VDC-SL-C:SRD-05VDC-SL-C K2
+U 1 1 600B249A
+P 6000 3400
+F 0 "K2" H 6000 3767 50  0000 C CNN
+F 1 "SRD-05VDC-SL-C" H 6000 3676 50  0000 C CNN
+F 2 "SRD-05VDC-SL-C:RELAY_SRD-05VDC-SL-C" H 6000 3400 50  0001 L BNN
+F 3 "" H 6000 3400 50  0001 L BNN
+F 4 "IPC-7251" H 6000 3400 50  0001 L BNN "STANDARD"
+F 5 "SONGLE RELAY" H 6000 3400 50  0001 L BNN "MANUFACTURER"
+	1    6000 3400
+	1    0    0    -1
+$EndComp
+$Comp
+L SRD-05VDC-SL-C:SRD-05VDC-SL-C K3
+U 1 1 600B35A7
+P 7800 3400
+F 0 "K3" H 7800 3767 50  0000 C CNN
+F 1 "SRD-05VDC-SL-C" H 7800 3676 50  0000 C CNN
+F 2 "SRD-05VDC-SL-C:RELAY_SRD-05VDC-SL-C" H 7800 3400 50  0001 L BNN
+F 3 "" H 7800 3400 50  0001 L BNN
+F 4 "IPC-7251" H 7800 3400 50  0001 L BNN "STANDARD"
+F 5 "SONGLE RELAY" H 7800 3400 50  0001 L BNN "MANUFACTURER"
+	1    7800 3400
+	1    0    0    -1
+$EndComp
 Wire Wire Line
-	7250 3250 7250 2750
-Connection ~ 7250 3250
-Connection ~ 7250 2750
+	7250 2750 7250 3300
 Wire Wire Line
-	7250 2750 6500 2750
+	5500 2750 6400 2750
+Wire Wire Line
+	5500 2750 5500 3300
+Wire Wire Line
+	3950 3300 3750 3300
+Connection ~ 3750 3300
+Wire Wire Line
+	3950 3600 3750 3600
+Connection ~ 3750 3600
+Wire Wire Line
+	4550 3300 4650 3300
+Wire Wire Line
+	4650 3300 4650 2750
+Connection ~ 4650 2750
+Wire Wire Line
+	4650 2750 5500 2750
+Wire Wire Line
+	6300 3300 6400 3300
+Wire Wire Line
+	6400 3300 6400 2750
+Connection ~ 6400 2750
+Wire Wire Line
+	6400 2750 7250 2750
+Wire Wire Line
+	7500 3300 7250 3300
+Connection ~ 7250 3300
+Wire Wire Line
+	7500 3600 7250 3600
+Connection ~ 7250 3600
+Wire Wire Line
+	8100 3300 8200 3300
+Wire Wire Line
+	8200 3300 8200 2750
+Wire Wire Line
+	8200 2750 7250 2750
+Wire Wire Line
+	5700 3600 5500 3600
+Connection ~ 5500 3600
+Wire Wire Line
+	5700 3300 5500 3300
+Connection ~ 5500 3300
 $EndSCHEMATC

Commit message: started pcb design
Parts:
- K1, K2, K3: symbol SRD-05VDC-SL-C:SRD-05VDC-SL-C -> plant-watering-rescue:SRD-05VDC-SL-C-SRD-05VDC-SL-C
Changed lines of the file:
@@
 Connection ~ 7250 2750
 $Comp
-L SRD-05VDC-SL-C:SRD-05VDC-SL-C K1
+L plant-watering-rescue:SRD-05VDC-SL-C-SRD-05VDC-SL-C K1
 U 1 1 600B0E95
 P 4250 3400
+AR Path="/600B0E95" Ref="K1"  Part="1"
+AR Path="/600A014F/600B0E95" Ref="K1"  Part="1"
 F 0 "K1" H 4250 3767 50  0000 C CNN
 F 1 "SRD-05VDC-SL-C" H 4250 3676 50  0000 C CNN
@@
 	3750 2750 4650 2750
 $Comp
-L SRD-05VDC-SL-C:SRD-05VDC-SL-C K2
+L plant-watering-rescue:SRD-05VDC-SL-C-SRD-05VDC-SL-C K2
 U 1 1 600B249A
 P 6000 3400
+AR Path="/600B249A" Ref="K2"  Part="1"
+AR Path="/600A014F/600B249A" Ref="K2"  Part="1"
 F 0 "K2" H 6000 3767 50  0000 C CNN
 F 1 "SRD-05VDC-SL-C" H 6000 3676 50  0000 C CNN
@@
 $EndComp
 $Comp
-L SRD-05VDC-SL-C:SRD-05VDC-SL-C K3
+L plant-watering-rescue:SRD-05VDC-SL-C-SRD-05VDC-SL-C K3
 U 1 1 600B35A7
 P 7800 3400
+AR Path="/600B35A7" Ref="K3"  Part="1"
+AR Path="/600A014F/600B35A7" Ref="K3"  Part="1"
 F 0 "K3" H 7800 3767 50  0000 C CNN
 F 1 "SRD-05VDC-SL-C" H 7800 3676 50  0000 C CNN

Commit message: added several parts#
Parts:
- added D4, D5, D6: D, Diodes_ThroughHole:D_DO-41_SOD81_P7.62mm_Horizontal, symbol Device:D
- added K4, K5, K6: SRD-05VDC-SL-C, SRD-05VDC-SL-C:RELAY_SRD-05VDC-SL-C, symbol plant-watering-rescue:SRD-05VDC-SL-C-SRD-05VDC-SL-C
Connections:
- net +5V: now also D4.1 (K), D5.1 (K), D6.1 (K), K4.A1, K4.NO, K5.A1, K5.NO, K6.A1, K6.NO
- new net M4: K4.COM
- new net M5: K5.COM
- new net M6: K6.COM
- new net RelayS4: D4.2 (A), K4.A2
- new net RelayS5: D5.2 (A), K5.A2
- new net RelayS6: D6.2 (A), K6.A2
Changed lines of the file:
@@
 $Descr A4 11693 8268
 encoding utf-8
-Sheet 5 6
+Sheet 5 7
 Title ""
 Date ""
@@
 	5700 3300 5500 3300
 Connection ~ 5500 3300
+$Comp
+L power:+5V #PWR0111
+U 1 1 6011430E
+P 3610 4200
+F 0 "#PWR0111" H 3610 4050 50  0001 C CNN
+F 1 "+5V" H 3625 4373 50  0000 C CNN
+F 2 "" H 3610 4200 50  0001 C CNN
+F 3 "" H 3610 4200 50  0001 C CNN
+	1    3610 4200
+	1    0    0    -1
+$EndComp
+Text GLabel 4560 4850 2    50   Input ~ 0
+M4
+Text GLabel 6310 4850 2    50   Input ~ 0
+M5
+Text GLabel 8110 4850 2    50   Input ~ 0
+M6
+Text GLabel 3760 5100 0    50   Input ~ 0
+RelayS4
+Text GLabel 5510 5100 0    50   Input ~ 0
+RelayS5
+Text GLabel 7260 5100 0    50   Input ~ 0
+RelayS6
+$Comp
+L Device:D D4
+U 1 1 6011431A
+P 3760 4900
+F 0 "D4" V 3714 4980 50  0000 L CNN
+F 1 "D" V 3805 4980 50  0000 L CNN
+F 2 "Diodes_ThroughHole:D_DO-41_SOD81_P7.62mm_Horizontal" H 3760 4900 50  0001 C CNN
+F 3 "~" H 3760 4900 50  0001 C CNN
+	1    3760 4900
+	0    1    1    0
+$EndComp
+$Comp
+L Device:D D5
+U 1 1 60114320
+P 5510 4900
+F 0 "D5" V 5464 4980 50  0000 L CNN
+F 1 "D" V 5555 4980 50  0000 L CNN
+F 2 "Diodes_ThroughHole:D_DO-41_SOD81_P7.62mm_Horizontal" H 5510 4900 50  0001 C CNN
+F 3 "~" H 5510 4900 50  0001 C CNN
+	1    5510 4900
+	0    1    1    0
+$EndComp
+$Comp
+L Device:D D6
+U 1 1 60114326
+P 7260 4900
+F 0 "D6" V 7214 4980 50  0000 L CNN
+F 1 "D" V 7305 4980 50  0000 L CNN
+F 2 "Diodes_ThroughHole:D_DO-41_SOD81_P7.62mm_Horizontal" H 7260 4900 50  0001 C CNN
+F 3 "~" H 7260 4900 50  0001 C CNN
+	1    7260 4900
+	0    1    1    0
+$EndComp
+Wire Wire Line
+	3760 5050 3760 5100
+Wire Wire Line
+	5510 5050 5510 5100
+Wire Wire Line
+	7260 5050 7260 5100
+Connection ~ 3760 4200
+Wire Wire Line
+	3760 4200 3610 4200
+Connection ~ 5510 4200
+Connection ~ 7260 4200
+$Comp
+L plant-watering-rescue:SRD-05VDC-SL-C-SRD-05VDC-SL-C K?
+U 1 1 60114335
+P 4260 4850
+AR Path="/60114335" Ref="K?"  Part="1"
+AR Path="/600A014F/60114335" Ref="K4"  Part="1"
+F 0 "K4" H 4260 5217 50  0000 C CNN
+F 1 "SRD-05VDC-SL-C" H 4260 5126 50  0000 C CNN
+F 2 "SRD-05VDC-SL-C:RELAY_SRD-05VDC-SL-C" H 4260 4850 50  0001 L BNN
+F 3 "" H 4260 4850 50  0001 L BNN
+F 4 "IPC-7251" H 4260 4850 50  0001 L BNN "STANDARD"
+F 5 "SONGLE RELAY" H 4260 4850 50  0001 L BNN "MANUFACTURER"
+	1    4260 4850
+	1    0    0    -1
+$EndComp
+Wire Wire Line
+	3760 4200 3760 4750
+Wire Wire Line
+	3760 4200 4660 4200
+$Comp
+L plant-watering-rescue:SRD-05VDC-SL-C-SRD-05VDC-SL-C K?
+U 1 1 6011433F
+P 6010 4850
+AR Path="/6011433F" Ref="K?"  Part="1"
+AR Path="/600A014F/6011433F" Ref="K5"  Part="1"
+F 0 "K5" H 6010 5217 50  0000 C CNN
+F 1 "SRD-05VDC-SL-C" H 6010 5126 50  0000 C CNN
+F 2 "SRD-05VDC-SL-C:RELAY_SRD-05VDC-SL-C" H 6010 4850 50  0001 L BNN
+F 3 "" H 6010 4850 50  0001 L BNN
+F 4 "IPC-7251" H 6010 4850 50  0001 L BNN "STANDARD"
+F 5 "SONGLE RELAY" H 6010 4850 50  0001 L BNN "MANUFACTURER"
+	1    6010 4850
+	1    0    0    -1
+$EndComp
+$Comp
+L plant-watering-rescue:SRD-05VDC-SL-C-SRD-05VDC-SL-C K?
+U 1 1 60114347
+P 7810 4850
+AR Path="/60114347" Ref="K?"  Part="1"
+AR Path="/600A014F/60114347" Ref="K6"  Part="1"
+F 0 "K6" H 7810 5217 50  0000 C CNN
+F 1 "SRD-05VDC-SL-C" H 7810 5126 50  0000 C CNN
+F 2 "SRD-05VDC-SL-C:RELAY_SRD-05VDC-SL-C" H 7810 4850 50  0001 L BNN
+F 3 "" H 7810 4850 50  0001 L BNN
+F 4 "IPC-7251" H 7810 4850 50  0001 L BNN "STANDARD"
+F 5 "SONGLE RELAY" H 7810 4850 50  0001 L BNN "MANUFACTURER"
+	1    7810 4850
+	1    0    0    -1
+$EndComp
+Wire Wire Line
+	7260 4200 7260 4750
+Wire Wire Line
+	5510 4200 6410 4200
+Wire Wire Line
+	5510 4200 5510 4750
+Wire Wire Line
+	3960 4750 3760 4750
+Connection ~ 3760 4750
+Wire Wire Line
+	3960 5050 3760 5050
+Connection ~ 3760 5050
+Wire Wire Line
+	4560 4750 4660 4750
+Wire Wire Line
+	4660 4750 4660 4200
+Connection ~ 4660 4200
+Wire Wire Line
+	4660 4200 5510 4200
+Wire Wire Line
+	6310 4750 6410 4750
+Wire Wire Line
+	6410 4750 6410 4200
+Connection ~ 6410 4200
+Wire Wire Line
+	6410 4200 7260 4200
+Wire Wire Line
+	7510 4750 7260 4750
+Connection ~ 7260 4750
+Wire Wire Line
+	7510 5050 7260 5050
+Connection ~ 7260 5050
+Wire Wire Line
+	8110 4750 8210 4750
+Wire Wire Line
+	8210 4750 8210 4200
+Wire Wire Line
+	8210 4200 7260 4200
+Wire Wire Line
+	5710 5050 5510 5050
+Connection ~ 5510 5050
+Wire Wire Line
+	5710 4750 5510 4750
+Connection ~ 5510 4750
 $EndSCHEMATC
