File: plant-watering/Input.sch (KiCad schematic (older format))
At the start: 2 parts, among them J4 Screw_Terminal_01x02

Commit message: changed transistor and relay circuit
Parts:
- removed C1: C, symbol Device:C
- removed J4: Screw_Terminal_01x02, Terminal_Blocks:TerminalBlock_bornier-2_P5.08mm, symbol Connector:Screw_Terminal_01x02
- added J?: USB_B_Micro, symbol Connector:USB_B_Micro
Connections:
- wire segments 8 -> 3
Changed lines of the file:
@@
 $EndDescr
-$Comp
-L Connector:Screw_Terminal_01x02 J4
-U 1 1 6009B47C
-P 5750 3550
-F 0 "J4" H 5830 3542 50  0000 L CNN
-F 1 "Screw_Terminal_01x02" H 5830 3451 50  0000 L CNN
-F 2 "Terminal_Blocks:TerminalBlock_bornier-2_P5.08mm" H 5750 3550 50  0001 C CNN
-F 3 "~" H 5750 3550 50  0001 C CNN
-	1    5750 3550
-	1    0    0    -1
-$EndComp
-$Comp
-L Device:C C1
-U 1 1 6009C312
-P 4850 3600
-F 0 "C1" H 4965 3646 50  0000 L CNN
-F 1 "C" H 4965 3555 50  0000 L CNN
-F 2 "" H 4888 3450 50  0001 C CNN
-F 3 "~" H 4850 3600 50  0001 C CNN
-	1    4850 3600
-	1    0    0    -1
-$EndComp
-Wire Wire Line
-	5550 3550 5550 3450
-Wire Wire Line
-	5550 3450 4850 3450
-Wire Wire Line
-	5550 3650 5550 3750
-Wire Wire Line
-	5550 3750 4850 3750
-Wire Wire Line
-	4850 3750 4850 3850
-Wire Wire Line
-	4850 3850 4700 3850
-Connection ~ 4850 3750
-Wire Wire Line
-	4850 3450 4850 3350
-Wire Wire Line
-	4850 3350 4700 3350
-Connection ~ 4850 3450
 $Comp
 L power:GND #PWR0103
 U 1 1 6009D169
-P 4700 3850
-F 0 "#PWR0103" H 4700 3600 50  0001 C CNN
-F 1 "GND" H 4705 3677 50  0000 C CNN
-F 2 "" H 4700 3850 50  0001 C CNN
-F 3 "" H 4700 3850 50  0001 C CNN
-	1    4700 3850
+P 4700 3990
+F 0 "#PWR0103" H 4700 3740 50  0001 C CNN
+F 1 "GND" H 4705 3817 50  0000 C CNN
+F 2 "" H 4700 3990 50  0001 C CNN
+F 3 "" H 4700 3990 50  0001 C CNN
+	1    4700 3990
 	1    0    0    -1
 $EndComp
@@
 	1    0    0    -1
 $EndComp
+$Comp
+L Connector:USB_B_Micro J?
+U 1 1 600B00AC
+P 3920 3590
+F 0 "J?" H 3977 4057 50  0000 C CNN
+F 1 "USB_B_Micro" H 3977 3966 50  0000 C CNN
+F 2 "" H 4070 3540 50  0001 C CNN
+F 3 "~" H 4070 3540 50  0001 C CNN
+	1    3920 3590
+	1    0    0    -1
+$EndComp
+Wire Wire Line
+	4220 3390 4700 3390
+Wire Wire Line
+	4700 3390 4700 3350
+Wire Wire Line
+	3920 3990 4700 3990
 $EndSCHEMATC

Commit message: edited schematic & started pcb design
Parts:
- removed J?: USB_B_Micro, symbol Connector:USB_B_Micro
- added J4: Input, Terminal_Blocks:TerminalBlock_bornier-2_P5.08mm, symbol Connector:Screw_Terminal_01x02
Changed lines of the file:
@@
 L power:GND #PWR0103
 U 1 1 6009D169
-P 4700 3990
-F 0 "#PWR0103" H 4700 3740 50  0001 C CNN
-F 1 "GND" H 4705 3817 50  0000 C CNN
-F 2 "" H 4700 3990 50  0001 C CNN
-F 3 "" H 4700 3990 50  0001 C CNN
-	1    4700 3990
+P 4450 3700
+F 0 "#PWR0103" H 4450 3450 50  0001 C CNN
+F 1 "GND" H 4455 3527 50  0000 C CNN
+F 2 "" H 4450 3700 50  0001 C CNN
+F 3 "" H 4450 3700 50  0001 C CNN
+	1    4450 3700
 	1    0    0    -1
 $EndComp
 $Comp
-L power:+5V #PWR0104
-U 1 1 6009D723
-P 4700 3350
-F 0 "#PWR0104" H 4700 3200 50  0001 C CNN
-F 1 "+5V" H 4715 3523 50  0000 C CNN
-F 2 "" H 4700 3350 50  0001 C CNN
-F 3 "" H 4700 3350 50  0001 C CNN
-	1    4700 3350
-	1    0    0    -1
+L Connector:Screw_Terminal_01x02 J4
+U 1 1 600BDABD
+P 3800 3700
+F 0 "J4" H 3718 3375 50  0000 C CNN
+F 1 "Input" H 3718 3466 50  0000 C CNN
+F 2 "Terminal_Blocks:TerminalBlock_bornier-2_P5.08mm" H 3800 3700 50  0001 C CNN
+F 3 "~" H 3800 3700 50  0001 C CNN
+	1    3800 3700
+	-1   0    0    1
 $EndComp
 $Comp
-L Connector:USB_B_Micro J?
-U 1 1 600B00AC
-P 3920 3590
-F 0 "J?" H 3977 4057 50  0000 C CNN
-F 1 "USB_B_Micro" H 3977 3966 50  0000 C CNN
-F 2 "" H 4070 3540 50  0001 C CNN
-F 3 "~" H 4070 3540 50  0001 C CNN
-	1    3920 3590
+L power:+5V #PWR0104
+U 1 1 600BEB7A
+P 4450 3550
+F 0 "#PWR0104" H 4450 3400 50  0001 C CNN
+F 1 "+5V" H 4465 3723 50  0000 C CNN
+F 2 "" H 4450 3550 50  0001 C CNN
+F 3 "" H 4450 3550 50  0001 C CNN
+	1    4450 3550
 	1    0    0    -1
 $EndComp
 Wire Wire Line
-	4220 3390 4700 3390
+	4000 3600 4450 3600
 Wire Wire Line
-	4700 3390 4700 3350
+	4450 3600 4450 3550
 Wire Wire Line
-	3920 3990 4700 3990
+	4000 3700 4450 3700
 $EndSCHEMATC

Commit message: changed pcb parts
Parts:
- J4: footprint Terminal_Blocks:TerminalBlock_bornier-2_P5.08mm -> TerminalBlock:TerminalBlock_Altech_AK300-2_P5.00mm
Changed lines of the file:
@@
 F 0 "J4" H 3718 3375 50  0000 C CNN
 F 1 "Input" H 3718 3466 50  0000 C CNN
-F 2 "Terminal_Blocks:TerminalBlock_bornier-2_P5.08mm" H 3800 3700 50  0001 C CNN
+F 2 "TerminalBlock:TerminalBlock_Altech_AK300-2_P5.00mm" H 3800 3700 50  0001 C CNN
 F 3 "~" H 3800 3700 50  0001 C CNN
 	1    3800 3700

Commit message: changed parts on pcb
Parts:
- J4: footprint TerminalBlock:TerminalBlock_Altech_AK300-2_P5.00mm -> TerminalBlock:ScrewTerminal_1x2_P5.00
Changed lines of the file:
@@
 F 0 "J4" H 3718 3375 50  0000 C CNN
 F 1 "Input" H 3718 3466 50  0000 C CNN
-F 2 "TerminalBlock:TerminalBlock_Altech_AK300-2_P5.00mm" H 3800 3700 50  0001 C CNN
+F 2 "TerminalBlock:ScrewTerminal_1x2_P5.00" H 3800 3700 50  0001 C CNN
 F 3 "~" H 3800 3700 50  0001 C CNN
 	1    3800 3700
