File: plant-watering/Input.sch (KiCad schematic (older format))
At the start: 2 parts, among them J4 Input

Commit message: forgot to save
Parts:
- C1: value CP -> 100uF
Changed lines of the file:
@@
 P 4820 3650
 F 0 "C1" H 4938 3696 50  0000 L CNN
-F 1 "CP" H 4938 3605 50  0000 L CNN
+F 1 "100uF" H 4938 3605 50  0000 L CNN
 F 2 "Capacitors_ThroughHole:CP_Radial_D6.3mm_P2.50mm" H 4858 3500 50  0001 C CNN
 F 3 "~" H 4820 3650 50  0001 C CNN
