File: plant-watering/UltrasonicSen.sch (KiCad schematic (older format))
At the start: 1 part, among them J14 Conn_01x04_Female

Commit message: changed pcb parts
Parts:
- J14: footprint Pin_Headers:Pin_Header_Straight_1x04_Pitch2.54mm -> TerminalBlock:TerminalBlock_Altech_AK300-4_P5.00mm
Changed lines of the file:
@@
 F 0 "J14" H 5028 2776 50  0000 L CNN
 F 1 "Conn_01x04_Female" H 5028 2685 50  0000 L CNN
-F 2 "Pin_Headers:Pin_Header_Straight_1x04_Pitch2.54mm" H 5000 2800 50  0001 C CNN
+F 2 "TerminalBlock:TerminalBlock_Altech_AK300-4_P5.00mm" H 5000 2800 50  0001 C CNN
 F 3 "~" H 5000 2800 50  0001 C CNN
 	1    5000 2800

Commit message: changed parts on pcb
Parts:
- J14: footprint TerminalBlock:TerminalBlock_Altech_AK300-4_P5.00mm -> TerminalBlock:ScrewTerminal_1x4_P5.00
Changed lines of the file:
@@
 F 0 "J14" H 5028 2776 50  0000 L CNN
 F 1 "Conn_01x04_Female" H 5028 2685 50  0000 L CNN
-F 2 "TerminalBlock:TerminalBlock_Altech_AK300-4_P5.00mm" H 5000 2800 50  0001 C CNN
+F 2 "TerminalBlock:ScrewTerminal_1x4_P5.00" H 5000 2800 50  0001 C CNN
 F 3 "~" H 5000 2800 50  0001 C CNN
 	1    5000 2800
