File: plant-watering/plant-watering.kicad_pcb (KiCad board)
At the start: 2 copper layers, 24 parts, among them J1 Conn_01x03_Male, J14 Conn_01x04_Female, J2 Conn_01x03_Male, J3 Conn_01x03_Male, J4 Input, J5 Screw_Terminal_01x08, J8 Conn_01x03_Male, K1 SRD-05VDC-SL-C, K2 SRD-05VDC-SL-C, K3 SRD-05VDC-SL-C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

Commit message: finished pcb for now
Parts:
- added REF**: MountingHole_3.2mm_M3_Pad_Via, Mounting_Holes:MountingHole_3.2mm_M3_Pad_Via, F.Cu at (91.4, 101.6)
- added REF**: MountingHole_3.2mm_M3_Pad_Via, Mounting_Holes:MountingHole_3.2mm_M3_Pad_Via, F.Cu at (165.1, 101.6)
- added REF**: MountingHole_3.2mm_M3_Pad_Via, Mounting_Holes:MountingHole_3.2mm_M3_Pad_Via, F.Cu at (91.4, 31.8)
- added REF**: MountingHole_3.2mm_M3_Pad_Via, Mounting_Holes:MountingHole_3.2mm_M3_Pad_Via, F.Cu at (165.1, 31.8)
- moved R4 94.6 mm to (123.2, 29.2), turned to 270 degrees
- moved Q4 92.8 mm to (123.2, 45.7), turned to 90 degrees
- moved J2 92.7 mm to (133.3, 30.5), turned to 90 degrees
- moved J4 88.1 mm to (91.4, 82.5)
- moved Q3 83.7 mm to (123.2, 66.0), turned to 90 degrees
- moved Q1 77.1 mm to (123.2, 106.7), turned to 90 degrees
- moved J8 74.7 mm to (165.1, 58.4)
- moved Q2 73.7 mm to (123.2, 86.4), turned to 90 degrees
- moved J1 71.8 mm to (153.7, 102.9), turned to 270 degrees
- moved J3 70.8 mm to (165.1, 77.5)
- moved U1 69.0 mm to (143.5, 67.3), turned to 180 degrees
- moved R3 67.9 mm to (123.2, 49.5), turned to 270 degrees
- moved K4 64.8 mm to (109.2, 35.6)
- moved J5 63.6 mm to (91.4, 80.0), turned to 180 degrees
- moved R2 50.0 mm to (123.2, 69.8), turned to 270 degrees
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Connections:
- U1 pad 10: Net-(U1-Pad10) -> GPIO26
Routing:
- net +5V: track 0.00 -> 173.0 mm
- net +3V3: track 0.00 -> 94.1 mm
- net GPIO12: track 0.00 -> 55.8 mm
- net GPIO33: track 0.00 -> 42.1 mm, vias 0 -> 1
- net GPIO13: track 0.00 -> 40.6 mm
- net GPIO16: track 0.00 -> 34.0 mm
- net GPIO34: track 0.00 -> 33.2 mm
- net GPIO32: track 0.00 -> 28.6 mm
- net M1: track 0.00 -> 25.5 mm
- net RelayS1: track 0.00 -> 24.6 mm
- net RelayS3: track 0.00 -> 24.6 mm
- net RelayS2: track 0.00 -> 24.6 mm
- net RelayS4: track 0.00 -> 24.6 mm
- net GPIO27: track 0.00 -> 20.3 mm
- net GPIO26: track 0.00 -> 20.1 mm
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- added copper zone on B.Cu, net GND
Other:
- board outline added: 88.9 x 87.6 mm

Commit message: added missing route
Routing:
- net +3V3: track 94.1 -> 114.7 mm
