File: plant-watering/plant-watering.kicad_pcb (KiCad board)
At the start: 2 copper layers, 88.9 x 87.6 mm, 28 parts, among them J1 Conn_01x03_Male, J14 Conn_01x04_Female, J2 Conn_01x03_Male, J3 Conn_01x03_Male, J4 Input, J5 Screw_Terminal_01x08, J8 Conn_01x03_Male, K1 SRD-05VDC-SL-C, K2 SRD-05VDC-SL-C, K3 SRD-05VDC-SL-C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

Commit message: added missing text
Other:
- board text added: "+"
- board text added: "-"
- board text added: "3V"
- board text added: "5-10k"
- board text added: "ESPHome-Plant-Watering"
- board text added: "INPUT 5V⎓2A"
- board text added: "IO26"
- board text added: "IO27"
- board text added: "IO32"
- board text added: "IO33"
- board text added: "IO34"
- board text added: "IO35"
- board text added: "MoiSen"
- board text added: "designed by Björn Ellwert"
