File: plant-watering/plant-watering.kicad_pcb (KiCad board)
At the start: 2 copper layers, 88.9 x 87.6 mm, 28 parts, among them J1 Conn_01x03_Male, J14 Conn_01x04_Female, J2 Conn_01x03_Male, J3 Conn_01x03_Male, J4 Input, J5 Screw_Terminal_01x08, J8 Conn_01x03_Male, K1 SRD-05VDC-SL-C, K2 SRD-05VDC-SL-C, K3 SRD-05VDC-SL-C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

Commit message: changed smth. finished and ordered
Parts:
- added C1: 100uF, Capacitors_ThroughHole:CP_Radial_D6.3mm_P2.50mm, F.Cu at (92.5, 81.8)
- moved J4 0.96 mm to (91.2, 83.5)
Routing:
- net +5V: track 173.0 -> 184.8 mm
Other:
- board text added: "IO12"
- board text added: "IO13"
- board text added: "IO16"
- board text added: "IO17"
